File: et-ruler-LitAC.kicad_sch (KiCad schematic)
At the start: 27 parts, among them J1 Conn_01x03, J2 AudioJack2, J3 Pmod-Interface-GPIO6, J4 Pmod-Interface-GPIO6, SW1 SW_DPDT, U1 OP07

Commit message: Add audio jack, links to parts, more footprints
Parts:
- D3: footprint LED_THT:LED_D5.0mm_Clear -> LED_HYBRID-emt:LED_THT_SMD_Hybrid_D5.0mm
- J1: footprint (none) -> Connector_PinSocket_2.54mm:PinSocket_1x03_P2.54mm_Vertical; now left out of the parts list
- J2: footprint (none) -> Connector_Audio:Jack_3.5mm_Ledino_KB3SPRS_Horizontal; Reichelt (none) -> https://www.reichelt.de/klinkeneinbaubuchse-3-5-mm-stereo-e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
- LS1: footprint (none) -> Connector_PinSocket_2.54mm:PinSocket_1x02_P2.54mm_Horizontal
- QR1: footprint et-ruler-footprints:QR-Code_15x15 -> Symbol-emt:qr-studiere-et_15x16
- RV1: Reichelt (none) -> https://www.reichelt.de/einstellpotentiometer-liegend-5-0-k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
Changed lines of the file:
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@@
   )
   (symbol (lib_id "Connector_Generic:Conn_01x03") (at 43.18 53.34 0) (unit 1)
-    (in_bom yes) (on_board yes) (fields_autoplaced)
+    (in_bom no) (on_board yes) (fields_autoplaced)
     (property "Reference" "J1" (id 0) (at 45.72 52.0699 0)
       (effects (font (size 1.27 1.27)) (justify left))
@@
       (effects (font (size 1.27 1.27)) (justify left))
     )
-    (property "Footprint" "" (id 2) (at 43.18 53.34 0)
+    (property "Footprint" "Connector_PinSocket_2.54mm:PinSocket_1x03_P2.54mm_Vertical" (id 2) (at 43.18 53.34 0)
       (effects (font (size 1.27 1.27)) hide)
     )
@@
       (effects (font (size 1.27 1.27)) (justify left))
     )
-    (property "Footprint" "LED_THT:LED_D5.0mm_Clear" (id 2) (at 80.01 111.76 0)
+    (property "Footprint" "LED_HYBRID-emt:LED_THT_SMD_Hybrid_D5.0mm" (id 2) (at 80.01 111.76 0)
       (effects (font (size 1.27 1.27)) hide)
     )
@@
       (effects (font (size 1.27 1.27)) (justify left))
     )
-    (property "Footprint" "et-ruler-footprints:QR-Code_15x15" (id 2) (at 97.79 57.785 0)
+    (property "Footprint" "Symbol-emt:qr-studiere-et_15x16" (id 2) (at 97.79 57.785 0)
       (effects (font (size 1.27 1.27)) hide)
     )
@@
       (effects (font (size 1.27 1.27)) (justify right))
     )
-    (property "Footprint" "" (id 2) (at 177.8 118.11 0)
+    (property "Footprint" "Connector_Audio:Jack_3.5mm_Ledino_KB3SPRS_Horizontal" (id 2) (at 177.8 118.11 0)
       (effects (font (size 1.27 1.27)) hide)
     )
     (property "Datasheet" "~" (id 3) (at 177.8 118.11 0)
+      (effects (font (size 1.27 1.27)) hide)
+    )
+    (property "Reichelt" "https://www.reichelt.de/klinkeneinbaubuchse-3-5-mm-stereo-ebs-35-p7301.html?&trstct=pos_0&nbc=1" (id 4) (at 177.8 118.11 0)
       (effects (font (size 1.27 1.27)) hide)
     )
@@
       (effects (font (size 1.27 1.27)) hide)
     )
+    (property "Reichelt" "https://www.reichelt.de/einstellpotentiometer-liegend-5-0-kohm-14-mm-acp-14-l-5k-p110274.html?&trstct=vrt_pdn&nbc=1" (id 4) (at 157.48 105.41 90)
+      (effects (font (size 1.27 1.27)) hide)
+    )
     (pin "1")
     (pin "2")
@@
       (effects (font (size 1.27 1.27)) (justify left))
     )
-    (property "Footprint" "" (id 2) (at 177.8 110.49 0)
+    (property "Footprint" "Connector_PinSocket_2.54mm:PinSocket_1x02_P2.54mm_Horizontal" (id 2) (at 177.8 110.49 0)
       (effects (font (size 1.27 1.27)) hide)
     )
@@
     )
     (path "/3f612082-f78a-4fc6-b4be-582c5a946fe6"
-      (reference "D3") (unit 1) (value "D_Photo") (footprint "LED_THT:LED_D5.0mm_Clear")
+      (reference "D3") (unit 1) (value "D_Photo") (footprint "LED_HYBRID-emt:LED_THT_SMD_Hybrid_D5.0mm")
     )
     (path "/46269970-1f41-4f51-a6e9-823721351469"
@@
     )
     (path "/1b629551-6b9c-438a-a71b-555bba6a38a8"
-      (reference "J1") (unit 1) (value "Conn_01x03") (footprint "")
+      (reference "J1") (unit 1) (value "Conn_01x03") (footprint "Connector_PinSocket_2.54mm:PinSocket_1x03_P2.54mm_Vertical")
     )
     (path "/6bd42537-1769-423f-b89f-3db96fb6df12"
-      (reference "J2") (unit 1) (value "AudioJack2") (footprint "")
+      (reference "J2") (unit 1) (value "AudioJack2") (footprint "Connector_Audio:Jack_3.5mm_Ledino_KB3SPRS_Horizontal")
     )
     (path "/65a0f130-acf5-437d-8d47-6972c0b0439e"
@@
     )
     (path "/d64f91a8-3ea7-4953-95c3-350cf0c6c3db"
-      (reference "LS1") (unit 1) (value "Speaker") (footprint "")
+      (reference "LS1") (unit 1) (value "Speaker") (footprint "Connector_PinSocket_2.54mm:PinSocket_1x02_P2.54mm_Horizontal")
     )
     (path "/619d303e-20a4-4608-a89a-df0d63123a33"
-      (reference "QR1") (unit 1) (value "QR ETrules") (footprint "et-ruler-footprints:QR-Code_15x15")
+      (reference "QR1") (unit 1) (value "QR ETrules") (footprint "Symbol-emt:qr-studiere-et_15x16")
     )
     (path "/c06bea49-d80e-472d-9d97-905f514fe83d"
