File: et-ruler-LitAC.kicad_sch (KiCad schematic)
At the start: 27 parts, among them J1 Conn_01x03, J2 AudioJack2, J3 Pmod-Interface-GPIO6, J4 Pmod-Interface-GPIO6, SW1 SW_DPDT, U1 OP07

Commit message: Exclude scales, holes, and logos from BOM
Parts:
- G1, G2, H1, H2, QR1, UniLogo1: now left out of the parts list
Changed lines of the file:
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@@
   )
   (symbol (lib_id "Mechanical:MountingHole") (at 97.79 38.1 0) (unit 1)
-    (in_bom yes) (on_board yes) (fields_autoplaced)
+    (in_bom no) (on_board yes) (fields_autoplaced)
     (property "Reference" "H2" (id 0) (at 100.33 36.8299 0)
       (effects (font (size 1.27 1.27)) (justify left))
@@
   )
   (symbol (lib_id "et-ruler-symbols:Ruler") (at 127 25.4 0) (unit 1)
-    (in_bom yes) (on_board yes) (fields_autoplaced)
+    (in_bom no) (on_board yes) (fields_autoplaced)
     (property "Reference" "G2" (id 0) (at 135.89 24.1299 0)
       (effects (font (size 1.27 1.27)) (justify left))
@@
   )
   (symbol (lib_id "Graphic:SYM_Flash_Small") (at 97.79 46.99 0) (unit 1)
-    (in_bom yes) (on_board yes)
+    (in_bom no) (on_board yes)
     (property "Reference" "UniLogo1" (id 0) (at 101.0412 45.6946 0)
       (effects (font (size 1.27 1.27)) (justify left))
@@
   )
   (symbol (lib_id "Mechanical:MountingHole") (at 97.79 33.02 0) (unit 1)
-    (in_bom yes) (on_board yes) (fields_autoplaced)
+    (in_bom no) (on_board yes) (fields_autoplaced)
     (property "Reference" "H1" (id 0) (at 100.33 31.7499 0)
       (effects (font (size 1.27 1.27)) (justify left))
@@
   )
   (symbol (lib_id "Graphic:SYM_Flash_Small") (at 97.79 57.15 0) (unit 1)
-    (in_bom yes) (on_board yes)
+    (in_bom no) (on_board yes)
     (property "Reference" "QR1" (id 0) (at 101.0158 55.8546 0)
       (effects (font (size 1.27 1.27)) (justify left))
@@
   )
   (symbol (lib_id "et-ruler-symbols:Ruler") (at 104.14 25.4 0) (unit 1)
-    (in_bom yes) (on_board yes) (fields_autoplaced)
+    (in_bom no) (on_board yes) (fields_autoplaced)
     (property "Reference" "G1" (id 0) (at 113.03 24.1299 0)
       (effects (font (size 1.27 1.27)) (justify left))

Commit message: Connect amplified signal to pmod
Connections:
- net amp_out: now reaches J2.S, LS1.1, R4.2, RV1.3
- net amp_out: now also J4.1 (IO1)
- no-connect marks 8 -> 7
Other:
- note added: "Output"
- moved on the sheet: J2, LS1
Changed lines of the file:
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@@
   (junction (at 113.03 88.9) (diameter 0) (color 0 0 0 0)
   )
+  (junction (at 224.79 102.87) (diameter 0) (color 0 0 0 0)
+  )
+  (junction (at 227.33 90.17) (diameter 0) (color 0 0 0 0)
+  )
   (junction (at 163.83 105.41) (diameter 0) (color 0 0 0 0)
   )
@@
   )
   (junction (at 149.86 105.41) (diameter 0) (color 0 0 0 0)
-  )
-  (junction (at 166.37 118.11) (diameter 0) (color 0 0 0 0)
-  )
-  (junction (at 168.91 105.41) (diameter 0) (color 0 0 0 0)
   )
   (junction (at 36.83 31.75) (diameter 0) (color 0 0 0 0)
@@
   (no_connect (at 215.9 30.48))
   (no_connect (at 187.96 44.45))
-  (no_connect (at 215.9 27.94))
   (no_connect (at 187.96 49.53))
+  (wire (pts (xy 215.9 27.94) (xy 218.44 27.94))
+    (stroke (width 0) (type default) (color 0 0 0 0))
+  )
   (polyline (pts (xy 93.98 66.04) (xy 147.32 66.04))
     (stroke (width 0) (type default) (color 0 0 0 0))
@@
     (stroke (width 0) (type default) (color 0 0 0 0))
   )
+  (polyline (pts (xy 198.12 129.54) (xy 266.7 129.54))
+    (stroke (width 0) (type default) (color 0 0 0 0))
+  )
   (polyline (pts (xy 194.31 129.54) (xy 194.31 69.85))
     (stroke (width 0) (type default) (color 0 0 0 0))
@@
     (stroke (width 0) (type default) (color 0 0 0 0))
   )
+  (wire (pts (xy 220.98 90.17) (xy 227.33 90.17))
+    (stroke (width 0) (type default) (color 0 0 0 0))
+  )
   (polyline (pts (xy 151.13 66.04) (xy 229.87 66.04))
     (stroke (width 0) (type default) (color 0 0 0 0))
@@
     (stroke (width 0) (type default) (color 0 0 0 0))
   )
-  (wire (pts (xy 166.37 118.11) (xy 172.72 118.11))
+  (wire (pts (xy 224.79 102.87) (xy 231.14 102.87))
     (stroke (width 0) (type default) (color 0 0 0 0))
   )
@@
     (stroke (width 0) (type default) (color 0 0 0 0))
   )
+  (polyline (pts (xy 198.12 69.85) (xy 266.7 69.85))
+    (stroke (width 0) (type default) (color 0 0 0 0))
+  )
   (wire (pts (xy 152.4 105.41) (xy 153.67 105.41))
     (stroke (width 0) (type default) (color 0 0 0 0))
@@
     (stroke (width 0) (type default) (color 0 0 0 0))
   )
-  (wire (pts (xy 168.91 105.41) (xy 172.72 105.41))
+  (wire (pts (xy 227.33 90.17) (xy 231.14 90.17))
     (stroke (width 0) (type default) (color 0 0 0 0))
   )
@@
     (stroke (width 0) (type default) (color 0 0 0 0))
   )
+  (polyline (pts (xy 198.12 69.85) (xy 198.12 129.54))
+    (stroke (width 0) (type default) (color 0 0 0 0))
+  )
   (wire (pts (xy 62.23 30.48) (xy 58.42 30.48))
     (stroke (width 0) (type default) (color 0 0 0 0))
@@
     (stroke (width 0) (type default) (color 0 0 0 0))
   )
-  (wire (pts (xy 166.37 107.95) (xy 166.37 118.11))
+  (wire (pts (xy 224.79 92.71) (xy 224.79 102.87))
     (stroke (width 0) (type default) (color 0 0 0 0))
   )
@@
     (stroke (width 0) (type default) (color 0 0 0 0))
   )
+  (polyline (pts (xy 266.7 129.54) (xy 266.7 69.85))
+    (stroke (width 0) (type default) (color 0 0 0 0))
+  )
   (polyline (pts (xy 17.78 17.78) (xy 91.44 17.78))
     (stroke (width 0) (type default) (color 0 0 0 0))
@@
     (stroke (width 0) (type default) (color 0 0 0 0))
   )
+  (wire (pts (xy 227.33 100.33) (xy 227.33 90.17))
+    (stroke (width 0) (type default) (color 0 0 0 0))
+  )
   (wire (pts (xy 135.89 105.41) (xy 140.97 105.41))
     (stroke (width 0) (type default) (color 0 0 0 0))
   )
-  (wire (pts (xy 168.91 115.57) (xy 172.72 115.57))
+  (wire (pts (xy 227.33 100.33) (xy 231.14 100.33))
     (stroke (width 0) (type default) (color 0 0 0 0))
   )
@@
     (stroke (width 0) (type default) (color 0 0 0 0))
   )
-  (wire (pts (xy 166.37 107.95) (xy 172.72 107.95))
+  (wire (pts (xy 224.79 92.71) (xy 231.14 92.71))
     (stroke (width 0) (type default) (color 0 0 0 0))
   )
@@
     (stroke (width 0) (type default) (color 0 0 0 0))
   )
-  (wire (pts (xy 166.37 118.11) (xy 166.37 120.65))
+  (wire (pts (xy 224.79 102.87) (xy 224.79 105.41))
     (stroke (width 0) (type default) (color 0 0 0 0))
   )
@@
   )
   (wire (pts (xy 26.67 55.88) (xy 26.67 53.34))
-    (stroke (width 0) (type default) (color 0 0 0 0))
-  )
-  (wire (pts (xy 168.91 105.41) (xy 168.91 115.57))
     (stroke (width 0) (type default) (color 0 0 0 0))
   )
@@
   )
   (text "Pmod connectors" (at 152.4 21.59 0)
+    (effects (font (size 2 2)) (justify left bottom))
+  )
+  (text "Output" (at 199.39 73.66 0)
     (effects (font (size 2 2)) (justify left bottom))
   )
@@
     )
   )
+  (global_label "amp_out" (shape input) (at 220.98 90.17 180) (fields_autoplaced)
+    (effects (font (size 1.27 1.27)) (justify right))
+    (property "Intersheet References" "${INTERSHEET_REFS}" (id 0) (at 210.584 90.0906 0)
+      (effects (font (size 1.27 1.27)) (justify right) hide)
+    )
+  )
   (global_label "V-" (shape input) (at 35.56 55.88 180) (fields_autoplaced)
     (effects (font (size 1.27 1.27)) (justify right))
@@
     (property "Intersheet References" "${INTERSHEET_REFS}" (id 0) (at 46.8145 39.2906 0)
       (effects (font (size 1.27 1.27)) (justify right) hide)
+    )
+  )
+  (global_label "amp_out" (shape input) (at 168.91 105.41 0) (fields_autoplaced)
+    (effects (font (size 1.27 1.27)) (justify left))
+    (property "Intersheet References" "${INTERSHEET_REFS}" (id 0) (at 179.306 105.4894 0)
+      (effects (font (size 1.27 1.27)) (justify left) hide)
+    )
+  )
+  (global_label "amp_out" (shape input) (at 218.44 27.94 0) (fields_autoplaced)
+    (effects (font (size 1.27 1.27)) (justify left))
+    (property "Intersheet References" "${INTERSHEET_REFS}" (id 0) (at 228.836 28.0194 0)
+      (effects (font (size 1.27 1.27)) (justify left) hide)
     )
   )
@@
     (pin "1")
   )
-  (symbol (lib_id "power:GND") (at 166.37 120.65 0) (unit 1)
-    (in_bom yes) (on_board yes)
-    (property "Reference" "#PWR07" (id 0) (at 166.37 127 0)
-      (effects (font (size 1.27 1.27)) hide)
-    )
-    (property "Value" "GND" (id 1) (at 166.497 125.0442 0))
-    (property "Footprint" "" (id 2) (at 166.37 120.65 0)
-      (effects (font (size 1.27 1.27)) hide)
-    )
-    (property "Datasheet" "" (id 3) (at 166.37 120.65 0)
+  (symbol (lib_id "power:GND") (at 224.79 105.41 0) (unit 1)
+    (in_bom yes) (on_board yes)
+    (property "Reference" "#PWR07" (id 0) (at 224.79 111.76 0)
+      (effects (font (size 1.27 1.27)) hide)
+    )
+    (property "Value" "GND" (id 1) (at 224.917 109.8042 0))
+    (property "Footprint" "" (id 2) (at 224.79 105.41 0)
+      (effects (font (size 1.27 1.27)) hide)
+    )
+    (property "Datasheet" "" (id 3) (at 224.79 105.41 0)
       (effects (font (size 1.27 1.27)) hide)
     )
@@
     (pin "1")
   )
-  (symbol (lib_id "Connector:AudioJack2") (at 177.8 118.11 0) (mirror y) (unit 1)
-    (in_bom yes) (on_board yes) (fields_autoplaced)
-    (property "Reference" "J2" (id 0) (at 182.88 116.2049 0)
+  (symbol (lib_id "Connector:AudioJack2") (at 236.22 102.87 0) (mirror y) (unit 1)
+    (in_bom yes) (on_board yes) (fields_autoplaced)
+    (property "Reference" "J2" (id 0) (at 241.3 100.9649 0)
       (effects (font (size 1.27 1.27)) (justify right))
     )
-    (property "Value" "AudioJack2" (id 1) (at 182.88 118.7449 0)
+    (property "Value" "AudioJack2" (id 1) (at 241.3 103.5049 0)
       (effects (font (size 1.27 1.27)) (justify right))
     )
-    (property "Footprint" "Connector_Audio:Jack_3.5mm_Ledino_KB3SPRS_Horizontal" (id 2) (at 177.8 118.11 0)
-      (effects (font (size 1.27 1.27)) hide)
-    )
-    (property "Datasheet" "~" (id 3) (at 177.8 118.11 0)
-      (effects (font (size 1.27 1.27)) hide)
-    )
-    (property "Reichelt" "https://www.reichelt.de/klinkeneinbaubuchse-3-5-mm-stereo-ebs-35-p7301.html?&trstct=pos_0&nbc=1" (id 4) (at 177.8 118.11 0)
+    (property "Footprint" "Connector_Audio:Jack_3.5mm_Ledino_KB3SPRS_Horizontal" (id 2) (at 236.22 102.87 0)
+      (effects (font (size 1.27 1.27)) hide)
+    )
+    (property "Datasheet" "~" (id 3) (at 236.22 102.87 0)
+      (effects (font (size 1.27 1.27)) hide)
+    )
+    (property "Reichelt" "https://www.reichelt.de/klinkeneinbaubuchse-3-5-mm-stereo-ebs-35-p7301.html?&trstct=pos_0&nbc=1" (id 4) (at 236.22 102.87 0)
       (effects (font (size 1.27 1.27)) hide)
     )
@@
     (pin "2")
   )
-  (symbol (lib_id "Device:Speaker") (at 177.8 105.41 0) (unit 1)
-    (in_bom yes) (on_board yes) (fields_autoplaced)
-    (property "Reference" "LS1" (id 0) (at 182.88 105.4099 0)
-      (effects (font (size 1.27 1.27)) (justify left))
-    )
-    (property "Value" "Speaker" (id 1) (at 182.88 107.9499 0)
-      (effects (font (size 1.27 1.27)) (justify left))
-    )
-    (property "Footprint" "Connector_PinSocket_2.54mm:PinSocket_1x02_P2.54mm_Horizontal" (id 2) (at 177.8 110.49 0)
-      (effects (font (size 1.27 1.27)) hide)
-    )
-    (property "Datasheet" "~" (id 3) (at 177.546 106.68 0)
-      (effects (font (size 1.27 1.27)) hide)
-    )
+  (symbol (lib_id "Device:Speaker") (at 236.22 90.17 0) (unit 1)
+    (in_bom yes) (on_board yes) (fields_autoplaced)
+    (property "Reference" "LS1" (id 0) (at 241.3 90.1699 0)
+      (effects (font (size 1.27 1.27)) (justify left))
+    )
+    (property "Value" "Speaker" (id 1) (at 241.3 92.7099 0)
+      (effects (font (size 1.27 1.27)) (justify left))
+    )
+    (property "Footprint" "Connector_PinSocket_2.54mm:PinSocket_1x02_P2.54mm_Horizontal" (id 2) (at 236.22 95.25 0)
+      (effects (font (size 1.27 1.27)) hide)
+    )
+    (property "Datasheet" "~" (id 3) (at 235.966 91.44 0)
+      (effects (font (size 1.27 1.27)) hide)
+    )
